Commit message: modified params in inertial_macros & robot model

File: ros2-waywise_description/urdf/camera.xacro (robot description, xacro)
@@ -8,25 +8,20 @@
       <material name="silver"/>
     </visual>
-    <xacro:inertial_box mass="0.1" x="0.025" y="0.125" z="0.03">
-    <origin xyz="0 0 0" rpy="0 0 0"/>
-  </xacro:inertial_box>
+    <xacro:inertial_box mass="0.1" length="0.025" breadth="0.125" height="0.03">
+      <origin xyz="0 0 0" rpy="0 0 0"/>
+    </xacro:inertial_box>
   </link>
   <joint name="camera_joint" type="fixed">
-    <parent link="base_link"/>
+    <parent link="chassis_link"/>
     <child link="camera_link"/>
-    <origin xyz="0.155 0 ${base_height/2 + 0.05}" rpy="0 0 0"/>
-  </joint>
-  <link name="camera_link_optical"></link>
-  <joint name="camera_optical_joint" type="fixed">
-    <parent link="camera_link"/>
-    <child link="camera_link_optical"/>
-    <origin xyz="0 0 0" rpy="${-pi/2} 0 ${-pi/2}"/>
+    <origin xyz="0.155 0 ${chassis_height/2 + 0.015}" rpy="0 0 0"/>
   </joint>
   <gazebo reference="camera_link">
-    <material>Gazebo/Black</material>
+    <material>Gazebo/Silver</material>
     <sensor name="camera" type="camera">
       <pose> 0 0 0 0 0 0 </pose>
       <visualize>true</visualize>
       <update_rate>10</update_rate>
+      <topic>camera</topic>
       <camera>
         <horizontal_fov>1.089</horizontal_fov>

File: ros2-waywise_description/urdf/depth_camera.xacro (robot description, xacro)
@@ -1,42 +1,37 @@
 <?xml version="1.0"?>
 <robot xmlns:xacro="http://www.ros.org/wiki/xacro" >
-  <link name="camera_link">
+  <link name="depth_camera_link">
     <visual>
       <geometry>
-        <box size="0.01 0.03 0.03"/>
+        <box size="0.025 0.125 0.03"/>
       </geometry>
-      <material name="red"/>
+      <material name="silver"/>
     </visual>
-    <xacro:inertial_box mass="0.1" x="0.01" y="0.03" z="0.03">
+    <xacro:inertial_box mass="0.1" length="0.025" breadth="0.125" height="0.03">
     <origin xyz="0 0 0" rpy="0 0 0"/>
   </xacro:inertial_box>
   </link>
-  <joint name="camera_joint" type="fixed">
-    <parent link="base_link"/>
-    <child link="camera_link"/>
-    <origin xyz="0.155 0 ${base_height/2 + 0.05}" rpy="0 0 0"/>
+  <joint name="depth_camera_joint" type="fixed">
+    <parent link="chassis_link"/>
+    <child link="depth_camera_link"/>
+    <origin xyz="0.155 0 ${chassis_height/2 + 0.015}" rpy="0 0 0"/>
   </joint>
-  <link name="camera_link_optical"></link>
-  <joint name="camera_optical_joint" type="fixed">
-    <parent link="camera_link"/>
-    <child link="camera_link_optical"/>
-    <origin xyz="0 0 0" rpy="${-pi/2} 0 ${-pi/2}"/>
-  </joint>
-  <gazebo reference="camera_link">
-    <material>Gazebo/Red</material>
-    <sensor name="camera" type="camera">
+  <gazebo reference="depth_camera_link">
+    <material>Gazebo/Silver</material>
+    <sensor name="depth_camera" type="depth_camera">
       <pose> 0 0 0 0 0 0 </pose>
+      <topic>depth_camera</topic>
       <visualize>true</visualize>
       <update_rate>10</update_rate>
       <camera>
-        <horizontal_fov>1.089</horizontal_fov>
+        <horizontal_fov>1.05</horizontal_fov>
         <image>
-          <format>R8G8B8</format>
-          <width>640</width>
-          <height>480</height>
+          <width>256</width>
+          <height>256</height>
+          <format>R_FLOAT32</format>
         </image>
         <clip>
-          <near>0.05</near>
-          <far>8.0</far>
+          <near>0.1</near>
+          <far>10.0</far>
         </clip>
       </camera>

File: ros2-waywise_description/urdf/imu.xacro (robot description, xacro)
@@ -13,12 +13,12 @@
       </geometry>
     </collision>
-    <xacro:inertial_box mass="0.1" x="0.075" y="0.075" z="0.02">
+    <xacro:inertial_box mass="0.1" length="0.075" breadth="0.075" height="0.02">
     <origin xyz="0 0 0" rpy="0 0 0"/>
   </xacro:inertial_box>
   </link>
   <joint name="imu_joint" type="fixed">
-    <parent link="base_link"/>
+    <parent link="chassis_link"/>
     <child link="imu_link"/>
-    <origin xyz="-0.08 0 ${base_height/2 + 0.01}"/>
+    <origin xyz="-0.08 0 ${chassis_height/2 + 0.01}"/>
   </joint>
   <gazebo reference="imu_link">

File: ros2-waywise_description/urdf/inertial_macros.xacro (robot description, xacro)
@@ -12,11 +12,11 @@
         </inertial>
     </xacro:macro>
-    <xacro:macro name="inertial_box" params="mass x y z *origin">
+    <xacro:macro name="inertial_box" params="mass length breadth height *origin">
         <inertial>
             <xacro:insert_block name="origin"/>
             <mass value="${mass}" />
-            <inertia ixx="${(1/12) * mass * (y*y+z*z)}" ixy="0.0" ixz="0.0"
-                    iyy="${(1/12) * mass * (x*x+z*z)}" iyz="0.0"
-                    izz="${(1/12) * mass * (x*x+y*y)}" />
+            <inertia ixx="${(1/12) * mass * (breadth*breadth+height*height)}" ixy="0.0" ixz="0.0"
+                    iyy="${(1/12) * mass * (length*length+height*height)}" iyz="0.0"
+                    izz="${(1/12) * mass * (length*length+breadth*breadth)}" />
         </inertial>
     </xacro:macro>

File: ros2-waywise_description/urdf/lidar.xacro (robot description, xacro)
@@ -1,15 +1,16 @@
 <?xml version="1.0"?>
 <robot xmlns:xacro="http://www.ros.org/wiki/xacro" >
-  <link name="lidar_frame">
+  <!-- Define lidar constants -->
+  <xacro:property name="lidar_mass" value="0.01"/>
+  <xacro:property name="lidar_support_mass" value="0.01"/>
+  <xacro:property name="lidar_radius" value="0.025"/>
+  <xacro:property name="lidar_length" value="0.03"/>
+  <xacro:property name="lidar_support_breadth" value="0.06"/>
+  <xacro:property name="lidar_support_length" value="0.06"/>
+  <xacro:property name="lidar_support_height" value="0.06"/>
+  <link name="lidar_link">
     <visual>
       <geometry>
-        <cylinder radius="0.025" length="0.03"/>
-      </geometry>
-      <material name="black"/>
-    </visual>
-    <visual>
-      <origin xyz="0 0 -0.05"/>
-      <geometry>
-        <cylinder radius="0.01" length="0.1"/>
+        <cylinder radius="${lidar_radius}" length="${lidar_length}"/>
       </geometry>
       <material name="black"/>
@@ -17,21 +18,45 @@
     <collision>
       <geometry>
-        <cylinder radius="0.025" length="0.03"/>
+        <cylinder radius="${lidar_radius}" length="${lidar_length}"/>
       </geometry>
     </collision>
-    <xacro:inertial_cylinder mass="0.01" length="0.025" radius="0.03">
+    <xacro:inertial_cylinder mass="${lidar_mass}" length="${lidar_length}" radius="${lidar_radius}">
       <origin xyz="0 0 0" rpy="0 0 0"/>
     </xacro:inertial_cylinder>
   </link>
+  <link name="lidar_support_link">
+    <visual>
+      <geometry>
+        <box size="${lidar_support_length} ${lidar_support_breadth} ${lidar_support_height}"/>
+      </geometry>
+      <material name="neon_blue"/>
+    </visual>
+    <collision>
+      <geometry>
+        <box size="${lidar_support_length} ${lidar_support_breadth} ${lidar_support_height}"/>
+      </geometry>
+    </collision>
+    <xacro:inertial_box mass="${lidar_mass}" length="${lidar_support_length}" breadth="${lidar_support_breadth}" height="${lidar_support_height}">
+      <origin xyz="0 0 0" rpy="0 0 0"/>
+    </xacro:inertial_box>
+  </link>
   <joint name="lidar_joint" type="fixed">
-    <parent link="base_link"/>
-    <child link="lidar_frame"/>
-    <origin xyz="0.11 0 ${base_height/2 + 0.095}" rpy="0 0 ${pi}"/>
+    <parent link="lidar_support_link"/>
+    <child link="lidar_link"/>
+    <origin xyz="0 0 ${lidar_length/2 + lidar_support_height/2}" rpy="0 0 0"/>
   </joint>
-  <gazebo reference="lidar_frame">
+  <joint name="lidar_support_joint" type="fixed">
+    <parent link="chassis_link"/>
+    <child link="lidar_support_link"/>
+    <origin xyz="0.12 0 ${chassis_height/2 + lidar_support_height/2}" rpy="0 0 0"/>
+  </joint>
+  <gazebo reference="lidar_link">
     <material>Gazebo/Black</material>
-    <sensor name='lidar' type='gpu_lidar'>"
-      <pose relative_to='lidar_frame'>0 0 0 0 0 0</pose>
-      <topic>lidar</topic>
+    <sensor name='lidar_link' type='gpu_lidar'>"
+      <topic>scan_lidar</topic>
+      <ignition_frame_id>lidar_link</ignition_frame_id>
+      <pose relative_to='lidar_link'>0 0 0 0 0 0</pose>
+      <always_on>true</always_on>
+      <visualize>false</visualize>
       <update_rate>10</update_rate>
       <ray>
@@ -40,10 +65,10 @@
             <samples>640</samples>
             <resolution>1</resolution>
-            <min_angle>-1.396263</min_angle>
-            <max_angle>1.396263</max_angle>
+            <min_angle>-3.1416</min_angle>
+            <max_angle>3.1416</max_angle>
           </horizontal>
           <vertical>
             <samples>1</samples>
-            <resolution>0.01</resolution>
+            <resolution>0.1</resolution>
             <min_angle>0</min_angle>
             <max_angle>0</max_angle>
@@ -51,11 +76,9 @@
         </scan>
         <range>
-          <min>0.08</min>
+          <min>0.20</min>
           <max>10.0</max>
-          <resolution>0.01</resolution>
+          <resolution>0.1</resolution>
         </range>
       </ray>
-      <alwaysOn>1</alwaysOn>
-      <visualize>true</visualize>
     </sensor>
   </gazebo>
