Commit message: added rplidar & updated lidar position in xacro

File: ros2-waywise_description/urdf/lidar.xacro (robot description, xacro)
@@ -44,5 +44,5 @@
     <parent link="lidar_support_link"/>
     <child link="lidar_link"/>
-    <origin xyz="0 0 ${lidar_length/2 + lidar_support_height/2}" rpy="0 0 0"/>
+    <origin xyz="0 0 ${lidar_length/2 + lidar_support_height/2}" rpy="0 0 ${pi}"/>
   </joint>
   <joint name="lidar_support_joint" type="fixed">
