Commit message: enable rgb and depth camera in robot.urdf.xacro and ros_gz_bridge

File: waywiser_description/urdf/camera.xacro (robot description, xacro)
@@ -1,27 +1,29 @@
 <?xml version="1.0"?>
-<robot xmlns:xacro="http://www.ros.org/wiki/xacro" >
+<robot xmlns:xacro="http://www.ros.org/wiki/xacro">
   <link name="camera_link">
     <visual>
       <geometry>
-        <box size="0.025 0.125 0.03"/>
+        <box size="0.025 0.125 0.03" />
       </geometry>
-      <material name="silver"/>
+      <material name="silver" />
     </visual>
     <xacro:inertial_box mass="0.1" length="0.025" breadth="0.125" height="0.03">
-      <origin xyz="0 0 0" rpy="0 0 0"/>
+      <origin xyz="0 0 0" rpy="0 0 0" />
     </xacro:inertial_box>
   </link>
   <joint name="camera_joint" type="fixed">
-    <parent link="chassis_link"/>
-    <child link="camera_link"/>
-    <origin xyz="0.155 0 ${chassis_height/2 + 0.015}" rpy="0 0 0"/>
+    <parent link="chassis_link" />
+    <child link="camera_link" />
+    <origin xyz="0.155 0 ${chassis_height/2 + 0.015}" rpy="0 0 0" />
   </joint>
   <gazebo reference="camera_link">
     <material>Gazebo/Silver</material>
     <sensor name="camera" type="camera">
-      <pose> 0 0 0 0 0 0 </pose>
-      <visualize>true</visualize>
-      <update_rate>10</update_rate>
-      <topic>camera</topic>
+      <always_on>1</always_on>
+      <visualize>0</visualize>
+      <update_rate>30</update_rate>
+      <topic>sensors/camera/image</topic>
+      <ignition_frame_id>camera_link</ignition_frame_id>
+      <pose relative_to='camera_link'>0 0 0 0 0 0</pose>
       <camera>
         <horizontal_fov>1.089</horizontal_fov>
@@ -33,5 +35,5 @@
         <clip>
           <near>0.05</near>
-          <far>8.0</far>
+          <far>30.0</far>
         </clip>
       </camera>

File: waywiser_description/urdf/depth_camera.xacro (robot description, xacro)
@@ -1,36 +1,42 @@
 <?xml version="1.0"?>
-<robot xmlns:xacro="http://www.ros.org/wiki/xacro" >
+<robot xmlns:xacro="http://www.ros.org/wiki/xacro">
   <link name="depth_camera_link">
     <visual>
       <geometry>
-        <box size="0.025 0.125 0.03"/>
+        <box size="0.025 0.125 0.03" />
       </geometry>
-      <material name="silver"/>
+      <material name="silver" />
     </visual>
     <xacro:inertial_box mass="0.1" length="0.025" breadth="0.125" height="0.03">
-    <origin xyz="0 0 0" rpy="0 0 0"/>
-  </xacro:inertial_box>
+      <origin xyz="0 0 0" rpy="0 0 0" />
+    </xacro:inertial_box>
   </link>
   <joint name="depth_camera_joint" type="fixed">
-    <parent link="chassis_link"/>
-    <child link="depth_camera_link"/>
-    <origin xyz="0.155 0 ${chassis_height/2 + 0.015}" rpy="0 0 0"/>
+    <parent link="chassis_link" />
+    <child link="depth_camera_link" />
+    <origin xyz="0.155 0 ${chassis_height/2 + 0.015}" rpy="0 0 0" />
   </joint>
   <gazebo reference="depth_camera_link">
     <material>Gazebo/Silver</material>
     <sensor name="depth_camera" type="depth_camera">
-      <pose> 0 0 0 0 0 0 </pose>
-      <topic>depth_camera</topic>
-      <visualize>true</visualize>
-      <update_rate>10</update_rate>
+      <always_on>1</always_on>
+      <visualize>0</visualize>
+      <update_rate>30</update_rate>
+      <topic>sensors/camera</topic>
+      <!-- <ignition_frame_id>depth_camera_link</ignition_frame_id> -->
+      <!-- A bug in depth_camera sensor does not allow setting frame_id for point clouds:
+      https://github.com/gazebosim/gz-sensors/pull/350 -->
+      <!-- It defaults to "robot/base_link/depth_camera" and can be handled either using a static
+      transformer or topic_tools-->
+      <pose relative_to='depth_camera_link'>0 0 0 0 0 0</pose>
       <camera>
-        <horizontal_fov>1.05</horizontal_fov>
+        <horizontal_fov>1.089</horizontal_fov>
         <image>
-          <width>256</width>
-          <height>256</height>
           <format>R_FLOAT32</format>
+          <width>640</width>
+          <height>480</height>
         </image>
         <clip>
-          <near>0.1</near>
+          <near>0.05</near>
           <far>10.0</far>
         </clip>

File: waywiser_description/urdf/robot.urdf.xacro (robot description, xacro)
@@ -9,6 +9,6 @@
     <xacro:include filename="lidar.xacro" />
     <xacro:include filename="imu.xacro" />
-    <!-- <xacro:include filename="camera.xacro" /> -->
-    <!--    <xacro:include filename="depth_camera.xacro" /> -->
+    <xacro:include filename="camera.xacro" />
+    <xacro:include filename="depth_camera.xacro" />
     <!-- Controller -->
     <xacro:if value="$(arg use_ros2_control)">

Commit message: feat: Update CMake configuration for C++20 and C23 standards, remove deprecated utility header, and enhance URDF/XACRO files for improved sensor integration and frame prefix support

File: waywiser_description/urdf/camera.xacro (robot description, xacro)
@@ -23,7 +23,7 @@
       <visualize>0</visualize>
       <update_rate>30</update_rate>
-      <topic>sensors/camera/image</topic>
-      <ignition_frame_id>camera_link</ignition_frame_id>
-      <pose relative_to='camera_link'>0 0 0 0 0 0</pose>
+      <topic>${robot_name}/sensors/camera/image</topic>
+      <ignition_frame_id>${robot_name}/camera_link</ignition_frame_id>
+      <pose relative_to='${robot_name}/camera_link'>0 0 0 0 0 0</pose>
       <camera>
         <horizontal_fov>1.089</horizontal_fov>

File: waywiser_description/urdf/gazebo_ackermann_control.xacro (robot description, xacro)
@@ -1,47 +1,59 @@
 <?xml version="1.0"?>
 <robot xmlns:xacro="http://www.ros.org/wiki/xacro">
-    <gazebo>
-      <plugin
-        filename="ignition-gazebo-ackermann-steering-system"
-        name="ignition::gazebo::systems::AckermannSteering">
-        <!-- Wheel Information -->
-        <left_joint>left_front_wheel_joint</left_joint>
-        <left_joint>left_rear_wheel_joint</left_joint>
-        <right_joint>right_front_wheel_joint</right_joint>
-        <right_joint>right_rear_wheel_joint</right_joint>
-        <left_steering_joint>left_front_wheel_steering_joint</left_steering_joint>
-        <right_steering_joint>right_front_wheel_steering_joint</right_steering_joint>
-        <wheel_separation>.21</wheel_separation>
-        <kingpin_width>.17</kingpin_width>
-        <steering_limit>0.5</steering_limit>
-        <steer_p_gain>1.0</steer_p_gain>
-        <wheel_base>.33</wheel_base>
-        <wheel_radius>0.055</wheel_radius>
-        <!-- Limits -->
-        <min_velocity>-100</min_velocity>
-        <max_velocity>100</max_velocity>
-        <min_acceleration>-5</min_acceleration>
-        <max_acceleration>5</max_acceleration>
-        <!-- Input -->
-        <topic>/cmd_vel</topic>
-        <!-- Output -->
-        <odom_publish_frequency>50</odom_publish_frequency>
-        <odom_topic>/odom</odom_topic>
-        <tf_topic>/tf</tf_topic>
-        <frame_id>odom</frame_id>
-        <child_frame_id>base_link</child_frame_id>
-      </plugin>
-    </gazebo>
-    <gazebo>
-      <plugin filename="libignition-gazebo-joint-state-publisher-system.so"
-        name="ignition::gazebo::systems::JointStatePublisher">
-        <joint_name>left_front_wheel_joint</joint_name>
-        <joint_name>left_rear_wheel_joint</joint_name>
-        <joint_name>right_front_wheel_joint</joint_name>
-        <joint_name>right_rear_wheel_joint</joint_name>
-        <joint_name>left_front_wheel_steering_joint</joint_name>
-        <joint_name>right_front_wheel_steering_joint</joint_name>
-        <topic>/joint_states</topic>
-      </plugin>
-    </gazebo>
+  <gazebo>
+    <plugin
+      filename="ignition-gazebo-ackermann-steering-system"
+      name="ignition::gazebo::systems::AckermannSteering">
+      <!-- Wheel Information -->
+      <left_joint>left_front_wheel_joint</left_joint>
+      <left_joint>left_rear_wheel_joint</left_joint>
+      <right_joint>right_front_wheel_joint</right_joint>
+      <right_joint>right_rear_wheel_joint</right_joint>
+      <left_steering_joint>left_front_wheel_steering_joint</left_steering_joint>
+      <right_steering_joint>right_front_wheel_steering_joint</right_steering_joint>
+      <wheel_separation>.21</wheel_separation>
+      <kingpin_width>.17</kingpin_width>
+      <steering_limit>0.5</steering_limit>
+      <steer_p_gain>1.0</steer_p_gain>
+      <wheel_base>.33</wheel_base>
+      <wheel_radius>0.055</wheel_radius>
+      <!-- Limits -->
+      <min_velocity>-100</min_velocity>
+      <max_velocity>100</max_velocity>
+      <min_acceleration>-5</min_acceleration>
+      <max_acceleration>5</max_acceleration>
+      <!-- Input -->
+      <topic>${robot_name}/cmd_vel</topic>
+      <!-- Output -->
+      <odom_publish_frequency>50</odom_publish_frequency>
+      <tf_topic>/tf</tf_topic>
+      <odom_topic>${robot_name}/odom</odom_topic>
+      <frame_id>${robot_name}/odom</frame_id>
+      <child_frame_id>${robot_name}/base_link</child_frame_id>
+    </plugin>
+  </gazebo>
+  <gazebo>
+    <plugin filename="libignition-gazebo-joint-state-publisher-system.so"
+      name="ignition::gazebo::systems::JointStatePublisher">
+      <joint_name>left_front_wheel_joint</joint_name>
+      <joint_name>left_rear_wheel_joint</joint_name>
+      <joint_name>right_front_wheel_joint</joint_name>
+      <joint_name>right_rear_wheel_joint</joint_name>
+      <joint_name>left_front_wheel_steering_joint</joint_name>
+      <joint_name>right_front_wheel_steering_joint</joint_name>
+      <topic>/joint_states</topic>
+    </plugin>
+    <plugin
+      filename="ignition-gazebo-pose-publisher-system"
+      name="gz::sim::systems::PosePublisher">
+      <publish_link_pose>false</publish_link_pose>
+      <publish_collision_pose>false</publish_collision_pose>
+      <publish_visual_pose>false</publish_visual_pose>
+      <publish_sensor_pose>false</publish_sensor_pose>
+      <publish_model_pose>true</publish_model_pose>
+      <use_pose_vector_msg>true</use_pose_vector_msg>
+      <publish_nested_model_pose>true</publish_nested_model_pose>
+      <update_frequency>50</update_frequency>
+    </plugin>
+  </gazebo>
 </robot>

File: waywiser_description/urdf/imu.xacro (robot description, xacro)
@@ -1,34 +1,34 @@
 <?xml version="1.0"?>
-<robot xmlns:xacro="http://www.ros.org/wiki/xacro" >
+<robot xmlns:xacro="http://www.ros.org/wiki/xacro">
   <link name="imu_link">
     <visual>
       <geometry>
-        <box size="0.075 0.075 0.02"/>
+        <box size="0.075 0.075 0.02" />
       </geometry>
-      <material name="black"/>
+      <material name="black" />
     </visual>
     <collision>
       <geometry>
-        <box size="0.075 0.075 0.2"/>
+        <box size="0.075 0.075 0.2" />
       </geometry>
     </collision>
     <xacro:inertial_box mass="0.1" length="0.075" breadth="0.075" height="0.02">
-    <origin xyz="0 0 0" rpy="0 0 0"/>
-  </xacro:inertial_box>
+      <origin xyz="0 0 0" rpy="0 0 0" />
+    </xacro:inertial_box>
   </link>
   <joint name="imu_joint" type="fixed">
-    <parent link="chassis_link"/>
-    <child link="imu_link"/>
-    <origin xyz="-0.08 0 ${chassis_height/2 + 0.01}"/>
+    <parent link="chassis_link" />
+    <child link="imu_link" />
+    <origin xyz="-0.08 0 ${chassis_height/2 + 0.01}" />
   </joint>
   <gazebo reference="imu_link">
     <material>Gazebo/Black</material>
     <sensor name="imu_sensor" type="imu">
-        <always_on>1</always_on>
-        <update_rate>30</update_rate>
-        <visualize>0</visualize>
-        <topic>imu</topic>
-        <ignition_frame_id>imu_link</ignition_frame_id>
-        <pose relative_to='imu_link'>0 0 0 0 0 0</pose>
+      <always_on>1</always_on>
+      <update_rate>30</update_rate>
+      <visualize>0</visualize>
+      <topic>${robot_name}/imu</topic>
+      <ignition_frame_id>${robot_name}/imu_link</ignition_frame_id>
+      <pose relative_to='${robot_name}/imu_link'>0 0 0 0 0 0</pose>
     </sensor>
   </gazebo>

File: waywiser_description/urdf/lidar.xacro (robot description, xacro)
@@ -2,25 +2,26 @@
 <robot xmlns:xacro="http://www.ros.org/wiki/xacro">
   <!-- Define lidar constants -->
-  <xacro:property name="lidar_mass" value="0.01"/>
-  <xacro:property name="lidar_support_mass" value="0.01"/>
-  <xacro:property name="lidar_radius" value="0.025"/>
-  <xacro:property name="lidar_length" value="0.03"/>
-  <xacro:property name="lidar_support_breadth" value="0.06"/>
-  <xacro:property name="lidar_support_length" value="0.06"/>
-  <xacro:property name="lidar_support_height" value="0.06"/>
+  <xacro:property name="lidar_mass" value="0.01" />
+  <xacro:property name="lidar_support_mass" value="0.01" />
+  <xacro:property name="lidar_radius" value="0.025" />
+  <xacro:property name="lidar_length" value="0.03" />
+  <xacro:property name="lidar_support_breadth" value="0.06" />
+  <xacro:property name="lidar_support_length" value="0.06" />
+  <xacro:property name="lidar_support_height" value="0.06" />
   <link name="lidar_link">
     <visual>
       <geometry>
-        <cylinder radius="${lidar_radius}" length="${lidar_length}"/>
+        <cylinder radius="${lidar_radius}" length="${lidar_length}" />
       </geometry>
-      <material name="black"/>
+      <material name="black" />
     </visual>
     <collision>
       <geometry>
-        <cylinder radius="${lidar_radius}" length="${lidar_length}"/>
+        <cylinder radius="${lidar_radius}" length="${lidar_length}" />
       </geometry>
     </collision>
-    <xacro:inertial_cylinder mass="${lidar_mass}" length="${lidar_length}" radius="${lidar_radius}">
-      <origin xyz="0 0 0" rpy="0 0 0"/>
+    <xacro:inertial_cylinder mass="${lidar_mass}" length="${lidar_length}"
+      radius="${lidar_radius}">
+      <origin xyz="0 0 0" rpy="0 0 0" />
     </xacro:inertial_cylinder>
   </link>
@@ -28,33 +29,34 @@
     <visual>
       <geometry>
-        <box size="${lidar_support_length} ${lidar_support_breadth} ${lidar_support_height}"/>
+        <box size="${lidar_support_length} ${lidar_support_breadth} ${lidar_support_height}" />
       </geometry>
-      <material name="neon_blue"/>
+      <material name="neon_blue" />
     </visual>
     <collision>
       <geometry>
-        <box size="${lidar_support_length} ${lidar_support_breadth} ${lidar_support_height}"/>
+        <box size="${lidar_support_length} ${lidar_support_breadth} ${lidar_support_height}" />
       </geometry>
     </collision>
-    <xacro:inertial_box mass="${lidar_mass}" length="${lidar_support_length}" breadth="${lidar_support_breadth}" height="${lidar_support_height}">
-      <origin xyz="0 0 0" rpy="0 0 0"/>
+    <xacro:inertial_box mass="${lidar_mass}" length="${lidar_support_length}"
+      breadth="${lidar_support_breadth}" height="${lidar_support_height}">
+      <origin xyz="0 0 0" rpy="0 0 0" />
     </xacro:inertial_box>
   </link>
   <joint name="lidar_joint" type="fixed">
-    <parent link="lidar_support_link"/>
-    <child link="lidar_link"/>
-    <origin xyz="0 0 ${lidar_length/2 + lidar_support_height/2}" rpy="0 0 ${pi}"/>
+    <parent link="lidar_support_link" />
+    <child link="lidar_link" />
+    <origin xyz="0 0 ${lidar_length/2 + lidar_support_height/2}" rpy="0 0 ${pi}" />
   </joint>
   <joint name="lidar_support_joint" type="fixed">
-    <parent link="chassis_link"/>
-    <child link="lidar_support_link"/>
-    <origin xyz="0.12 0 ${chassis_height/2 + lidar_support_height/2}" rpy="0 0 0"/>
+    <parent link="chassis_link" />
+    <child link="lidar_support_link" />
+    <origin xyz="0.12 0 ${chassis_height/2 + lidar_support_height/2}" rpy="0 0 0" />
   </joint>
   <gazebo reference="lidar_link">
     <material>Gazebo/Black</material>
-    <sensor name='lidar_link' type='gpu_lidar'>"
-      <topic>scan_lidar</topic>
-      <ignition_frame_id>lidar_link</ignition_frame_id>
-      <pose relative_to='lidar_link'>0 0 0 0 0 0</pose>
+    <sensor name='lidar_link' type='gpu_lidar'>
+      <topic>${robot_name}/scan_lidar</topic>
+      <ignition_frame_id>${robot_name}/lidar_link</ignition_frame_id>
+      <pose relative_to="${robot_name}/lidar_link">0 0 0 0 0 0</pose>
       <always_on>1</always_on>
       <visualize>0</visualize>

File: waywiser_description/urdf/realsense_d435i_camera.xacro (robot description, xacro)
@@ -64,7 +64,7 @@
       <visualize>0</visualize>
       <update_rate>30</update_rate>
-      <pose relative_to='camera_link'>0 0 0 0 0 0</pose>
-      <ignition_frame_id>camera_link</ignition_frame_id>
-      <topic>sensors/camera</topic>
+      <pose relative_to='${robot_name}/camera_link'>0 0 0 0 0 0</pose>
+      <ignition_frame_id>${robot_name}/camera_link</ignition_frame_id>
+      <topic>${robot_name}/sensors/camera</topic>
       <camera>
         <horizontal_fov>1.089</horizontal_fov>

File: waywiser_description/urdf/rover.urdf.xacro (robot description, xacro)
@@ -4,4 +4,7 @@
     <xacro:arg name="use_ros2_control" default="false" />
     <xacro:arg name="sim_mode" default="false" />
+    <xacro:arg name="robot_name" default="rover" />
+    <xacro:attribute name="name" value="$(arg robot_name)" />
+    <xacro:property name="robot_name" value="$(arg robot_name)" />
     <!-- Robot model without sensors -->
     <xacro:include filename="rover_core.xacro" />
@@ -12,4 +15,6 @@
     <!-- <xacro:include filename="depth_camera.xacro" /> -->
     <xacro:include filename="realsense_d435i_camera.xacro" />
+    <xacro:property name="gps_parent_link" value="chassis_link" />
+    <xacro:include filename="gps.xacro" />
     <!-- Controller -->
     <xacro:if value="$(arg use_ros2_control)">
