Commit message: feat: Update URDF and utility functions to support frame prefix handling, ensuring consistent topic and frame naming across various sensors and components.

File: waywiser_description/urdf/camera.xacro (robot description, xacro)
@@ -23,7 +23,7 @@
       <visualize>0</visualize>
       <update_rate>30</update_rate>
-      <topic>${robot_name}/sensors/camera/image</topic>
-      <ignition_frame_id>${robot_name}/camera_link</ignition_frame_id>
-      <pose relative_to='${robot_name}/camera_link'>0 0 0 0 0 0</pose>
+      <topic>${frame_prefix}sensors/camera/image</topic>
+      <ignition_frame_id>${frame_prefix}camera_link</ignition_frame_id>
+      <pose relative_to='${frame_prefix}camera_link'>0 0 0 0 0 0</pose>
       <camera>
         <horizontal_fov>1.089</horizontal_fov>

File: waywiser_description/urdf/gazebo_ackermann_control.xacro (robot description, xacro)
@@ -2,7 +2,5 @@
 <robot xmlns:xacro="http://www.ros.org/wiki/xacro">
   <gazebo>
-    <plugin
-      filename="ignition-gazebo-ackermann-steering-system"
-      name="ignition::gazebo::systems::AckermannSteering">
+    <plugin filename="ignition-gazebo-ackermann-steering-system" name="ignition::gazebo::systems::AckermannSteering">
       <!-- Wheel Information -->
       <left_joint>left_front_wheel_joint</left_joint>
@@ -24,16 +22,15 @@
       <max_acceleration>5</max_acceleration>
       <!-- Input -->
-      <topic>${robot_name}/cmd_vel</topic>
+      <topic>${frame_prefix}cmd_vel</topic>
       <!-- Output -->
       <odom_publish_frequency>50</odom_publish_frequency>
       <tf_topic>/tf</tf_topic>
-      <odom_topic>${robot_name}/odom</odom_topic>
-      <frame_id>${robot_name}/odom</frame_id>
-      <child_frame_id>${robot_name}/base_link</child_frame_id>
+      <odom_topic>${frame_prefix}odom</odom_topic>
+      <frame_id>${frame_prefix}odom</frame_id>
+      <child_frame_id>${frame_prefix}base_link</child_frame_id>
     </plugin>
   </gazebo>
   <gazebo>
-    <plugin filename="libignition-gazebo-joint-state-publisher-system.so"
-      name="ignition::gazebo::systems::JointStatePublisher">
+    <plugin filename="libignition-gazebo-joint-state-publisher-system.so" name="ignition::gazebo::systems::JointStatePublisher">
       <joint_name>left_front_wheel_joint</joint_name>
       <joint_name>left_rear_wheel_joint</joint_name>
@@ -44,7 +41,5 @@
       <topic>/joint_states</topic>
     </plugin>
-    <plugin
-      filename="ignition-gazebo-pose-publisher-system"
-      name="gz::sim::systems::PosePublisher">
+    <plugin filename="ignition-gazebo-pose-publisher-system" name="gz::sim::systems::PosePublisher">
       <publish_link_pose>false</publish_link_pose>
       <publish_collision_pose>false</publish_collision_pose>

File: waywiser_description/urdf/gps.xacro (robot description, xacro)
@@ -28,7 +28,7 @@
             <update_rate>10</update_rate>
             <visualize>0</visualize>
-            <topic>${robot_name}/gps/navsat</topic>
-            <ignition_frame_id>${robot_name}/gps_link</ignition_frame_id>
-            <pose relative_to='${robot_name}/gps_link'>0 0 0 0 0 0</pose>
+            <topic>${frame_prefix}gps/navsat</topic>
+            <ignition_frame_id>${frame_prefix}gps_link</ignition_frame_id>
+            <pose relative_to='${frame_prefix}gps_link'>0 0 0 0 0 0</pose>
             <navsat>
                 <position_sensing>

File: waywiser_description/urdf/imu.xacro (robot description, xacro)
@@ -28,7 +28,7 @@
       <update_rate>30</update_rate>
       <visualize>0</visualize>
-      <topic>${robot_name}/imu</topic>
-      <ignition_frame_id>${robot_name}/imu_link</ignition_frame_id>
-      <pose relative_to='${robot_name}/imu_link'>0 0 0 0 0 0</pose>
+      <topic>${frame_prefix}imu</topic>
+      <ignition_frame_id>${frame_prefix}imu_link</ignition_frame_id>
+      <pose relative_to='${frame_prefix}imu_link'>0 0 0 0 0 0</pose>
     </sensor>
   </gazebo>

File: waywiser_description/urdf/lidar.xacro (robot description, xacro)
@@ -21,6 +21,5 @@
       </geometry>
     </collision>
-    <xacro:inertial_cylinder mass="${lidar_mass}" length="${lidar_length}"
-      radius="${lidar_radius}">
+    <xacro:inertial_cylinder mass="${lidar_mass}" length="${lidar_length}" radius="${lidar_radius}">
       <origin xyz="0 0 0" rpy="0 0 0" />
     </xacro:inertial_cylinder>
@@ -38,6 +37,5 @@
       </geometry>
     </collision>
-    <xacro:inertial_box mass="${lidar_mass}" length="${lidar_support_length}"
-      breadth="${lidar_support_breadth}" height="${lidar_support_height}">
+    <xacro:inertial_box mass="${lidar_mass}" length="${lidar_support_length}" breadth="${lidar_support_breadth}" height="${lidar_support_height}">
       <origin xyz="0 0 0" rpy="0 0 0" />
     </xacro:inertial_box>
@@ -56,7 +54,7 @@
     <material>Gazebo/Black</material>
     <sensor name='lidar_link' type='gpu_lidar'>
-      <topic>${robot_name}/scan_lidar</topic>
-      <ignition_frame_id>${robot_name}/lidar_link</ignition_frame_id>
-      <pose relative_to="${robot_name}/lidar_link">0 0 0 0 0 0</pose>
+      <topic>${frame_prefix}scan_lidar</topic>
+      <ignition_frame_id>${frame_prefix}lidar_link</ignition_frame_id>
+      <pose relative_to="${frame_prefix}lidar_link">0 0 0 0 0 0</pose>
       <always_on>1</always_on>
       <visualize>0</visualize>

File: waywiser_description/urdf/realsense_d435i_camera.xacro (robot description, xacro)
@@ -7,13 +7,10 @@
       <origin xyz="0 0 0" rpy="0 0 1.570795" />
       <mass value="0.0615752" />
-      <inertia ixx="9.108e-05" ixy="0.0" ixz="0.0"
-        iyy="2.51e-06" iyz="0.0"
-        izz="8.931e-05" />
+      <inertia ixx="9.108e-05" ixy="0.0" ixz="0.0" iyy="2.51e-06" iyz="0.0" izz="8.931e-05" />
     </inertial>
     <collision name="collision">
       <origin xyz="0 0 0" rpy="0 0 1.570795" />
       <geometry>
-        <mesh
-          filename="package://waywiser_description/sdf/realsense_d435i_camera/meshes/realsense.dae">
+        <mesh filename="package://waywiser_description/sdf/realsense_d435i_camera/meshes/realsense.dae">
         </mesh>
       </geometry>
@@ -22,6 +19,5 @@
       <origin xyz="0 0 0" rpy="0 0 1.570795" />
       <geometry>
-        <mesh
-          filename="package://waywiser_description/sdf/realsense_d435i_camera/meshes/realsense.dae">
+        <mesh filename="package://waywiser_description/sdf/realsense_d435i_camera/meshes/realsense.dae">
           <submesh>
             <name>RealSense</name>
@@ -64,7 +60,7 @@
       <visualize>0</visualize>
       <update_rate>30</update_rate>
-      <pose relative_to='${robot_name}/camera_link'>0 0 0 0 0 0</pose>
-      <ignition_frame_id>${robot_name}/camera_link</ignition_frame_id>
-      <topic>${robot_name}/sensors/camera</topic>
+      <pose relative_to='${frame_prefix}camera_link'>0 0 0 0 0 0</pose>
+      <ignition_frame_id>${frame_prefix}camera_link</ignition_frame_id>
+      <topic>${frame_prefix}sensors/camera</topic>
       <camera>
         <horizontal_fov>1.089</horizontal_fov>

File: waywiser_description/urdf/rover.urdf.xacro (robot description, xacro)
@@ -4,7 +4,6 @@
     <xacro:arg name="use_ros2_control" default="false" />
     <xacro:arg name="sim_mode" default="false" />
-    <xacro:arg name="robot_name" default="rover" />
-    <xacro:attribute name="name" value="$(arg robot_name)" />
-    <xacro:property name="robot_name" value="$(arg robot_name)" />
+    <xacro:arg name="frame_prefix" default="/" />
+    <xacro:property name="frame_prefix" value="$(arg frame_prefix)" />
     <!-- Robot model without sensors -->
     <xacro:include filename="rover_core.xacro" />
